Commit message: Update manipulator urdf

File: alicia_duo_descriptions/urdf/alicia_duo_with_gripper.urdf (robot description, URDF)
Before this commit: robot alicia_duo_descriptions, 11 links, 10 joints
Links:
- link Grasp_base: mass 0.0482959693358257 -> 0.13604884360545
- link Link1: mass 0.1961 -> 0.203075737500143
- link Link2: mass 0.21717 -> 0.228750683078605
- link Link3: mass 0.0865602005421272 -> 0.0902084989642731
- link Link4: mass 0.0943760430662397 -> 0.0791974889780253
- link Link5: mass 0.0298054906363541 -> 0.0472226666291309
- link Link6: mass 0.00075405362358679 -> 0.000754043064008528
- link Link7: mass 0.0298800419940728 -> 0.0243492837152759
- link Link8: mass 0.0298800419940728 -> 0.0243228050977196
Joints:
- joint Grasp2tool: origin xyz=-0.0065308 -0.00063845 0.11382 rpy=0 0 0 -> xyz=0.00275 0.0008332 0.13779 rpy=0 0 0
- joint Joint1: origin xyz=0 0 0.0745 rpy=0 0 0 -> xyz=0 0 0.1445 rpy=0 0 0
- joint Joint2: origin xyz=-4E-05 0 0.09361 rpy=-1.5708 -1.4701 0 -> xyz=0 0 0.025106 rpy=1.5708 -1.5708 0
- joint Joint3: origin xyz=0.22471 0 0.0004 rpy=0 0 -2.4569 -> xyz=0.22367 0.022494 -5E-05 rpy=0 0 2.3562
- joint Joint4: origin xyz=0.00211 -0.0969 -0.0005 rpy=1.5708 0 0 -> xyz=0.0988 0.00211 -0.0001 rpy=1.5708 0 1.5708
- joint Joint5: origin xyz=0.00014 0.0002 0.12011 rpy=-1.5708 0 0 -> xyz=0 -0.0007 0.12011 rpy=-1.5708 0 0
- joint Joint6: origin xyz=-0.00389 -0.0592 0.00064 rpy=1.5708 0 0 -> xyz=-0.0038938 -0.0573 0.0008 rpy=1.5708 0 0
- joint left_finger: axis 0 0 -1 -> 0 0 0; limit (none) -> lower=-0.0125 upper=0 effort=5 velocity=10; origin xyz=-0.0065308 -0.015222 0.11382 rpy=1.5708 0 0 -> xyz=0.00275 -0.0011661 0.13779 rpy=1.5451 0 0
- joint right_finger: axis 0 0 1 -> 0 0 0; limit (none) -> lower=0 upper=0.0125 effort=5 velocity=10; origin xyz=-0.0065308 0.013945 0.11382 rpy=1.5708 0 3.1416 -> xyz=0.00275 0.0028325 0.13768 rpy=-1.5965 0 0
