Commit message: Update meshes dir

File: alicia_duo_descriptions/urdf/alicia_duo_with_gripper_v0.urdf (robot description, URDF)
Before this commit: robot alicia_D_v5_4_50mm_gripper, 11 links, 10 joints
Links:
- link Grasp_base: geometry collision mesh filename=package://alicia_duo_descriptions/meshes_v1/Grasp_base.STL; visual mesh filename=package://alicia_duo_descriptions/meshes_v1/Grasp_base.STL
- link Link1: geometry collision mesh filename=package://alicia_duo_descriptions/meshes_v1/Link1.STL; visual mesh filename=package://alicia_duo_descriptions/meshes_v1/Link1.STL
- link Link2: geometry collision mesh filename=package://alicia_duo_descriptions/meshes_v1/Link2.STL; visual mesh filename=package://alicia_duo_descriptions/meshes_v1/Link2.STL
- link Link3: geometry collision mesh filename=package://alicia_duo_descriptions/meshes_v1/Link3.STL; visual mesh filename=package://alicia_duo_descriptions/meshes_v1/Link3.STL
- link Link4: geometry collision mesh filename=package://alicia_duo_descriptions/meshes_v1/Link4.STL; visual mesh filename=package://alicia_duo_descriptions/meshes_v1/Link4.STL
- link Link5: geometry collision mesh filename=package://alicia_duo_descriptions/meshes_v1/Link5.STL; visual mesh filename=package://alicia_duo_descriptions/meshes_v1/Link5.STL
- link Link6: geometry collision mesh filename=package://alicia_duo_descriptions/meshes_v1/Link6.STL; visual mesh filename=package://alicia_duo_descriptions/meshes_v1/Link6.STL
- link Link7: geometry collision mesh filename=package://alicia_duo_descriptions/meshes_v1/Link7.STL; visual mesh filename=package://alicia_duo_descriptions/meshes_v1/Link7.STL
- link Link8: geometry collision mesh filename=package://alicia_duo_descriptions/meshes_v1/Link8.STL; visual mesh filename=package://alicia_duo_descriptions/meshes_v1/Link8.STL
- link base_link: geometry collision mesh filename=package://alicia_duo_descriptions/meshes_v1/base_link.STL; visual mesh filename=package://alicia_duo_descriptions/meshes_v1/base_link.STL

File: alicia_duo_descriptions/urdf/alicia_duo_with_gripper_v1.urdf (robot description, URDF)
Before this commit: robot alicia_D_v5_4_100mm_gripper, 11 links, 10 joints
Links:
- link Grasp_base: geometry collision mesh filename=package://alicia_duo_descriptions/meshes_v1/Grasp_base.STL; visual mesh filename=package://alicia_duo_descriptions/meshes_v1/Grasp_base.STL
- link Link1: geometry collision mesh filename=package://alicia_duo_descriptions/meshes_v1/Link1.STL; visual mesh filename=package://alicia_duo_descriptions/meshes_v1/Link1.STL
- link Link2: geometry collision mesh filename=package://alicia_duo_descriptions/meshes_v1/Link2.STL; visual mesh filename=package://alicia_duo_descriptions/meshes_v1/Link2.STL
- link Link3: geometry collision mesh filename=package://alicia_duo_descriptions/meshes_v1/Link3.STL; visual mesh filename=package://alicia_duo_descriptions/meshes_v1/Link3.STL
- link Link4: geometry collision mesh filename=package://alicia_duo_descriptions/meshes_v1/Link4.STL; visual mesh filename=package://alicia_duo_descriptions/meshes_v1/Link4.STL
- link Link5: geometry collision mesh filename=package://alicia_duo_descriptions/meshes_v1/Link5.STL; visual mesh filename=package://alicia_duo_descriptions/meshes_v1/Link5.STL
- link Link6: geometry collision mesh filename=package://alicia_duo_descriptions/meshes_v1/Link6.STL; visual mesh filename=package://alicia_duo_descriptions/meshes_v1/Link6.STL
- link Link7: geometry collision mesh filename=package://alicia_duo_descriptions/meshes_v1/Link7.STL; visual mesh filename=package://alicia_duo_descriptions/meshes_v1/Link7.STL
- link Link8: geometry collision mesh filename=package://alicia_duo_descriptions/meshes_v1/Link8.STL; visual mesh filename=package://alicia_duo_descriptions/meshes_v1/Link8.STL
- link base_link: geometry collision mesh filename=package://alicia_duo_descriptions/meshes_v1/base_link.STL; visual mesh filename=package://alicia_duo_descriptions/meshes_v1/base_link.STL
